File: GPSLoRa.sch (KiCad schematic (older format))
At the start: 48 parts, among them P1 IN EXT, P2 - INPUT 12 +, P3 OUT EXT, P4 Battery, P5 CONN_01X01, Q1 Q_NPN_BCE, SW1 SW_PUSH_OP, U1 4N26, U2 LM2596_Breakout, U3 4N26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

Commit message: Update kicad 4.0.5
Parts:
- D4, D5, D6, D7, D8: symbol LED -> LED-RESCUE-GPSLoRa
Changed lines of the file:
@@
 EESchema Schematic File Version 2
+LIBS:GPSLoRa-rescue
 LIBS:power
 LIBS:device
@@
 RST
 $Comp
-L GND #PWR2
+L GND #PWR01
 U 1 1 57EC269A
 P 1200 2050
-F 0 "#PWR2" H 1200 1800 50  0001 C CNN
+F 0 "#PWR01" H 1200 1800 50  0001 C CNN
 F 1 "GND" H 1200 1900 50  0000 C CNN
 F 2 "" H 1200 2050 50  0000 C CNN
@@
 $EndComp
 $Comp
-L GND #PWR10
+L GND #PWR02
 U 1 1 57EC26BA
 P 3400 1850
-F 0 "#PWR10" H 3400 1600 50  0001 C CNN
+F 0 "#PWR02" H 3400 1600 50  0001 C CNN
 F 1 "GND" H 3400 1700 50  0000 C CNN
 F 2 "" H 3400 1850 50  0000 C CNN
@@
 DIO0
 $Comp
-L GND #PWR21
+L GND #PWR03
 U 1 1 57EC27C1
 P 6390 2815
-F 0 "#PWR21" H 6390 2565 50  0001 C CNN
+F 0 "#PWR03" H 6390 2565 50  0001 C CNN
 F 1 "GND" H 6390 2665 50  0000 C CNN
 F 2 "" H 6390 2815 50  0000 C CNN
@@
 RX
 $Comp
-L GND #PWR34
+L GND #PWR04
 U 1 1 57EC2AF4
 P 10100 2750
-F 0 "#PWR34" H 10100 2500 50  0001 C CNN
+F 0 "#PWR04" H 10100 2500 50  0001 C CNN
 F 1 "GND" H 10100 2600 50  0000 C CNN
 F 2 "" H 10100 2750 50  0000 C CNN
@@
 NoConn ~ 2400 1200
 $Comp
-L GND #PWR24
+L GND #PWR05
 U 1 1 57EC3E17
 P 7490 1965
-F 0 "#PWR24" H 7490 1715 50  0001 C CNN
+F 0 "#PWR05" H 7490 1715 50  0001 C CNN
 F 1 "GND" H 7490 1815 50  0000 C CNN
 F 2 "" H 7490 1965 50  0000 C CNN
@@
 $EndComp
 $Comp
-L GND #PWR22
+L GND #PWR06
 U 1 1 57EC3EF2
 P 7040 2715
-F 0 "#PWR22" H 7040 2465 50  0001 C CNN
+F 0 "#PWR06" H 7040 2465 50  0001 C CNN
 F 1 "GND" H 7040 2565 50  0000 C CNN
 F 2 "" H 7040 2715 50  0000 C CNN
@@
 $EndComp
 $Comp
-L GND #PWR26
+L GND #PWR07
 U 1 1 57EC4654
 P 7795 2475
-F 0 "#PWR26" H 7795 2225 50  0001 C CNN
+F 0 "#PWR07" H 7795 2225 50  0001 C CNN
 F 1 "GND" H 7795 2325 50  0000 C CNN
 F 2 "" H 7795 2475 50  0000 C CNN
@@
 $EndComp
 $Comp
-L GND #PWR38
+L GND #PWR08
 U 1 1 57EC47A9
 P 10600 2350
-F 0 "#PWR38" H 10600 2100 50  0001 C CNN
+F 0 "#PWR08" H 10600 2100 50  0001 C CNN
 F 1 "GND" H 10600 2200 50  0000 C CNN
 F 2 "" H 10600 2350 50  0000 C CNN
@@
 $EndComp
 $Comp
-L GND #PWR27
+L GND #PWR09
 U 1 1 57EC470D
 P 8215 5070
-F 0 "#PWR27" H 8215 4820 50  0001 C CNN
+F 0 "#PWR09" H 8215 4820 50  0001 C CNN
 F 1 "GND" H 8215 4920 50  0000 C CNN
 F 2 "" H 8215 5070 50  0000 C CNN
@@
 $EndComp
 $Comp
-L +BATT #PWR31
+L +BATT #PWR010
 U 1 1 57EC48A4
 P 8765 4120
-F 0 "#PWR31" H 8765 3970 50  0001 C CNN
+F 0 "#PWR010" H 8765 3970 50  0001 C CNN
 F 1 "+BATT" H 8765 4260 50  0000 C CNN
 F 2 "" H 8765 4120 50  0000 C CNN
@@
 $EndComp
 $Comp
-L LED D4
+L LED-RESCUE-GPSLoRa D4
 U 1 1 57EC4E60
 P 5465 4520
@@
 $EndComp
 $Comp
-L LED D5
+L LED-RESCUE-GPSLoRa D5
 U 1 1 57EC4EE4
 P 5465 4820
@@
 $EndComp
 $Comp
-L GND #PWR9
+L GND #PWR011
 U 1 1 57EC56BB
 P 3250 4775
-F 0 "#PWR9" H 3250 4525 50  0001 C CNN
+F 0 "#PWR011" H 3250 4525 50  0001 C CNN
 F 1 "GND" H 3250 4625 50  0000 C CNN
 F 2 "" H 3250 4775 50  0000 C CNN
@@
 $EndComp
 $Comp
-L +5V #PWR14
+L +5V #PWR012
 U 1 1 57EC622A
 P 4450 4275
-F 0 "#PWR14" H 4450 4125 50  0001 C CNN
+F 0 "#PWR012" H 4450 4125 50  0001 C CNN
 F 1 "+5V" H 4450 4415 50  0000 C CNN
 F 2 "" H 4450 4275 50  0000 C CNN
@@
 $EndComp
 $Comp
-L +5V #PWR16
+L +5V #PWR013
 U 1 1 57EC6354
 P 4965 4220
-F 0 "#PWR16" H 4965 4070 50  0001 C CNN
+F 0 "#PWR013" H 4965 4070 50  0001 C CNN
 F 1 "+5V" H 4965 4360 50  0000 C CNN
 F 2 "" H 4965 4220 50  0000 C CNN
@@
 Jumper adjust voltage
 $Comp
-L +BATT #PWR8
+L +BATT #PWR014
 U 1 1 57F9BDBF
 P 3150 1600
-F 0 "#PWR8" H 3150 1450 50  0001 C CNN
+F 0 "#PWR014" H 3150 1450 50  0001 C CNN
 F 1 "+BATT" H 3150 1740 50  0000 C CNN
 F 2 "" H 3150 1600 50  0000 C CNN
@@
 D8
 $Comp
-L GND #PWR7
+L GND #PWR015
 U 1 1 580A553D
 P 2750 7495
-F 0 "#PWR7" H 2750 7245 50  0001 C CNN
+F 0 "#PWR015" H 2750 7245 50  0001 C CNN
 F 1 "GND" H 2750 7345 50  0000 C CNN
 F 2 "" H 2750 7495 50  0000 C CNN
@@
 $EndComp
 $Comp
-L GND #PWR13
+L GND #PWR016
 U 1 1 580EBBF8
 P 4100 7310
-F 0 "#PWR13" H 4100 7060 50  0001 C CNN
+F 0 "#PWR016" H 4100 7060 50  0001 C CNN
 F 1 "GND" H 4100 7160 50  0000 C CNN
 F 2 "" H 4100 7310 50  0000 C CNN
@@
 $EndComp
 $Comp
-L +BATT #PWR4
+L +BATT #PWR017
 U 1 1 580EC6C4
 P 1615 6195
-F 0 "#PWR4" H 1615 6045 50  0001 C CNN
+F 0 "#PWR017" H 1615 6045 50  0001 C CNN
 F 1 "+BATT" H 1615 6335 50  0000 C CNN
 F 2 "" H 1615 6195 50  0000 C CNN
@@
 $EndComp
 $Comp
-L +BATT #PWR11
+L +BATT #PWR018
 U 1 1 580EFD19
 P 3600 6365
-F 0 "#PWR11" H 3600 6215 50  0001 C CNN
+F 0 "#PWR018" H 3600 6215 50  0001 C CNN
 F 1 "+BATT" H 3600 6505 50  0000 C CNN
 F 2 "" H 3600 6365 50  0000 C CNN
@@
 $EndComp
 $Comp
-L +12C #PWR12
+L +12C #PWR019
 U 1 1 580EFE55
 P 4100 6300
-F 0 "#PWR12" H 4100 6150 50  0001 C CNN
+F 0 "#PWR019" H 4100 6150 50  0001 C CNN
 F 1 "+12C" H 4100 6450 50  0000 C CNN
 F 2 "" H 4100 6300 50  0000 C CNN
@@
 $EndComp
 $Comp
-L +12C #PWR1
+L +12C #PWR020
 U 1 1 580F036C
 P 800 6175
-F 0 "#PWR1" H 800 6025 50  0001 C CNN
+F 0 "#PWR020" H 800 6025 50  0001 C CNN
 F 1 "+12C" H 800 6325 50  0000 C CNN
 F 2 "" H 800 6175 50  0000 C CNN
@@
 $EndComp
 $Comp
-L GND #PWR5
+L GND #PWR021
 U 1 1 580F08E0
 P 1615 6855
-F 0 "#PWR5" H 1615 6605 50  0001 C CNN
+F 0 "#PWR021" H 1615 6605 50  0001 C CNN
 F 1 "GND" H 1615 6705 50  0000 C CNN
 F 2 "" H 1615 6855 50  0000 C CNN
@@
 $EndComp
 $Comp
-L +12C #PWR3
+L +12C #PWR022
 U 1 1 580EFF04
 P 1460 4370
-F 0 "#PWR3" H 1460 4220 50  0001 C CNN
+F 0 "#PWR022" H 1460 4220 50  0001 C CNN
 F 1 "+12C" H 1460 4520 50  0000 C CNN
 F 2 "" H 1460 4370 50  0000 C CNN
@@
 $EndComp
 $Comp
-L LED D6
+L LED-RESCUE-GPSLoRa D6
 U 1 1 583891C8
 P 7705 3280
@@
 $EndComp
 $Comp
-L GND #PWR23
+L GND #PWR023
 U 1 1 58389C04
 P 7280 3395
-F 0 "#PWR23" H 7280 3145 50  0001 C CNN
+F 0 "#PWR023" H 7280 3145 50  0001 C CNN
 F 1 "GND" H 7280 3245 50  0000 C CNN
 F 2 "" H 7280 3395 50  0000 C CNN
@@
 $EndComp
 $Comp
-L +BATT #PWR28
+L +BATT #PWR024
 U 1 1 5838A13A
 P 8445 3180
-F 0 "#PWR28" H 8445 3030 50  0001 C CNN
+F 0 "#PWR024" H 8445 3030 50  0001 C CNN
 F 1 "+BATT" H 8445 3320 50  0000 C CNN
 F 2 "" H 8445 3180 50  0000 C CNN
@@
 $EndComp
 $Comp
-L LED D7
+L LED-RESCUE-GPSLoRa D7
 U 1 1 58405E18
 P 2295 3445
@@
 $EndComp
 $Comp
-L GND #PWR6
+L GND #PWR025
 U 1 1 58405E27
 P 1870 3560
-F 0 "#PWR6" H 1870 3310 50  0001 C CNN
+F 0 "#PWR025" H 1870 3310 50  0001 C CNN
 F 1 "GND" H 1870 3410 50  0000 C CNN
 F 2 "" H 1870 3560 50  0000 C CNN
@@
 $EndComp
 $Comp
-L LED D8
+L LED-RESCUE-GPSLoRa D8
 U 1 1 58405F1A
 P 5105 3355
@@
 $EndComp
 $Comp
-L GND #PWR15
+L GND #PWR026
 U 1 1 58405F29
 P 4680 3470
-F 0 "#PWR15" H 4680 3220 50  0001 C CNN
+F 0 "#PWR026" H 4680 3220 50  0001 C CNN
 F 1 "GND" H 4680 3320 50  0000 C CNN
 F 2 "" H 4680 3470 50  0000 C CNN
@@
 NoConn ~ 5995 7240
 $Comp
-L +BATT #PWR18
+L +BATT #PWR027
 U 1 1 5841AD5D
 P 6095 6780
-F 0 "#PWR18" H 6095 6630 50  0001 C CNN
+F 0 "#PWR027" H 6095 6630 50  0001 C CNN
 F 1 "+BATT" H 6095 6920 50  0000 C CNN
 F 2 "" H 6095 6780 50  0000 C CNN
@@
 $EndComp
 $Comp
-L GND #PWR19
+L GND #PWR028
 U 1 1 5841AD70
 P 6095 7440
-F 0 "#PWR19" H 6095 7190 50  0001 C CNN
+F 0 "#PWR028" H 6095 7190 50  0001 C CNN
 F 1 "GND" H 6095 7290 50  0000 C CNN
 F 2 "" H 6095 7440 50  0000 C CNN
@@
 $EndComp
 $Comp
-L GND #PWR17
+L GND #PWR029
 U 1 1 5842104A
 P 5270 7495
-F 0 "#PWR17" H 5270 7245 50  0001 C CNN
+F 0 "#PWR029" H 5270 7245 50  0001 C CNN
 F 1 "GND" H 5270 7345 50  0000 C CNN
 F 2 "" H 5270 7495 50  0000 C CNN
@@
 $EndComp
 $Comp
-L GND #PWR39
+L GND #PWR030
 U 1 1 5842B8F0
 P 9915 4115
-F 0 "#PWR39" H 9915 3865 50  0001 C CNN
+F 0 "#PWR030" H 9915 3865 50  0001 C CNN
 F 1 "GND" H 9915 3965 50  0000 C CNN
 F 2 "" H 9915 4115 50  0000 C CNN
@@
 $EndComp
 $Comp
-L GND #PWR35
+L GND #PWR031
 U 1 1 5845EC29
 P 10255 5980
-F 0 "#PWR35" H 10255 5730 50  0001 C CNN
+F 0 "#PWR031" H 10255 5730 50  0001 C CNN
 F 1 "GND" H 10255 5830 50  0000 C CNN
 F 2 "" H 10255 5980 50  0000 C CNN
@@
 $EndComp
 $Comp
-L GND #PWR32
+L GND #PWR032
 U 1 1 5845ECCD
 P 9155 5895
-F 0 "#PWR32" H 9155 5645 50  0001 C CNN
+F 0 "#PWR032" H 9155 5645 50  0001 C CNN
 F 1 "GND" H 9155 5745 50  0000 C CNN
 F 2 "" H 9155 5895 50  0000 C CNN
@@
 $EndComp
 $Comp
-L GND #PWR30
+L GND #PWR033
 U 1 1 5845ED71
 P 8590 6055
-F 0 "#PWR30" H 8590 5805 50  0001 C CNN
+F 0 "#PWR033" H 8590 5805 50  0001 C CNN
 F 1 "GND" H 8590 5905 50  0000 C CNN
 F 2 "" H 8590 6055 50  0000 C CNN
@@
 NoConn ~ 9975 5825
 $Comp
-L +3.3V #PWR36
+L +3.3V #PWR034
 U 1 1 58460528
 P 10395 5565
-F 0 "#PWR36" H 10395 5415 50  0001 C CNN
+F 0 "#PWR034" H 10395 5415 50  0001 C CNN
 F 1 "+3.3V" H 10395 5705 50  0000 C CNN
 F 2 "" H 10395 5565 50  0000 C CNN
@@
 $EndComp
 $Comp
-L +BATT #PWR29
+L +BATT #PWR035
 U 1 1 584605CC
 P 8505 5570
-F 0 "#PWR29" H 8505 5420 50  0001 C CNN
+F 0 "#PWR035" H 8505 5420 50  0001 C CNN
 F 1 "+BATT" H 8505 5710 50  0000 C CNN
 F 2 "" H 8505 5570 50  0000 C CNN
@@
 $EndComp
 $Comp
-L +3.3V #PWR20
+L +3.3V #PWR036
 U 1 1 58461FEF
 P 6390 1615
-F 0 "#PWR20" H 6390 1465 50  0001 C CNN
+F 0 "#PWR036" H 6390 1465 50  0001 C CNN
 F 1 "+3.3V" H 6390 1755 50  0000 C CNN
 F 2 "" H 6390 1615 50  0000 C CNN
@@
 $EndComp
 $Comp
-L +3.3V #PWR37
+L +3.3V #PWR037
 U 1 1 5846263D
 P 10600 1900
-F 0 "#PWR37" H 10600 1750 50  0001 C CNN
+F 0 "#PWR037" H 10600 1750 50  0001 C CNN
 F 1 "+3.3V" H 10600 2040 50  0000 C CNN
 F 2 "" H 10600 1900 50  0000 C CNN
@@
 $EndComp
 $Comp
-L +3.3V #PWR25
+L +3.3V #PWR038
 U 1 1 58462C8B
 P 7795 2025
-F 0 "#PWR25" H 7795 1875 50  0001 C CNN
+F 0 "#PWR038" H 7795 1875 50  0001 C CNN
 F 1 "+3.3V" H 7795 2165 50  0000 C CNN
 F 2 "" H 7795 2025 50  0000 C CNN
@@
 $EndComp
 $Comp
-L +3.3V #PWR?
+L +3.3V #PWR039
 U 1 1 5850A43E
 P 10100 1400
-F 0 "#PWR?" H 10100 1250 50  0001 C CNN
+F 0 "#PWR039" H 10100 1250 50  0001 C CNN
 F 1 "+3.3V" H 10100 1540 50  0000 C CNN
 F 2 "" H 10100 1400 50  0000 C CNN
@@
 $EndComp
 $Comp
-L +3.3V #PWR?
+L +3.3V #PWR040
 U 1 1 5850DCED
 P 10705 4580
-F 0 "#PWR?" H 10705 4430 50  0001 C CNN
+F 0 "#PWR040" H 10705 4430 50  0001 C CNN
 F 1 "+3.3V" H 10705 4720 50  0000 C CNN
 F 2 "" H 10705 4580 50  0000 C CNN
