File: GPSLoRa.kicad_pcb (KiCad board)
At the start: 2 copper layers, 30 parts, among them P1 IN EXT, P2 - INPUT 12 +, P3 OUT EXT, P4 Battery, Q1 Q_NPN_BCE, U1 4N26, U2 LM2596_Breakout, U3 4N26, U4 RFM95W-868S2, U5 MCP73831T-2ATI/OT

Commit message: Added PCB 0.1v
Parts:
- moved D1 57.4 mm to (115.5, 95.0), turned to 180 degrees
- moved U1 53.0 mm to (119.9, 81.6), turned to 270 degrees
- moved D3 50.6 mm to (121.6, 94.7)
- moved P3 49.8 mm to (163.2, 102.5), turned to 180 degrees
- moved MODULE1 49.1 mm to (177.6, 64.9), turned to 180 degrees
- moved D4 47.8 mm to (114.2, 75.8), turned to 180 degrees
- moved R2 47.2 mm to (137.8, 86.7), turned to 180 degrees
- moved R9 45.7 mm to (129.7, 73.7)
- moved R1 44.6 mm to (137.8, 83.9), turned to 180 degrees
- moved D5 44.1 mm to (114.2, 73.3), turned to 180 degrees
- moved P1 42.7 mm to (155.8, 102.5)
- moved P4 40.9 mm to (178.2, 102.5), turned to 270 degrees
- moved R3 40.6 mm to (137.8, 81.2)
- moved uP1 40.0 mm to (117.6, 63.0), turned to 90 degrees
- moved R6 38.3 mm to (137.8, 89.4), turned to 180 degrees
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Routing:
- net +BATT: track 0.00 -> 209.9 mm
- net +5V: track 0.00 -> 131.2 mm, vias 0 -> 1
- net +12C: track 0.00 -> 85.7 mm, vias 0 -> 1
- net /RX: track 0.00 -> 76.5 mm, vias 0 -> 3
- net /TX: track 0.00 -> 70.4 mm, vias 0 -> 3
- net /D6: track 0.00 -> 64.2 mm
- net /SCK: track 0.00 -> 45.2 mm, vias 0 -> 1
- net Net-(D1-Pad1): track 0.00 -> 44.2 mm
- net /MISO: track 0.00 -> 42.7 mm, vias 0 -> 1
- net /MOSI: track 0.00 -> 38.6 mm, vias 0 -> 1
- net /NSS: track 0.00 -> 37.7 mm, vias 0 -> 2
- net Net-(D3-Pad2): track 0.00 -> 37.6 mm
- net Net-(R4-Pad2): track 0.00 -> 37.2 mm, vias 0 -> 2
- net /DIO0: track 0.00 -> 30.5 mm
- net /DIO1: track 0.00 -> 30.0 mm
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- added copper zone on B.Cu, net GND
- added copper zone on F.Cu, net GND
Other:
- board outline added: 80 x 55 mm
- net class Default: trace_width 0.25 -> 0.3
- net class Vcc added: clearance 0.2, trace_width 0.5, via_dia 0.8, via_drill 0.6

Commit message: Added logos
Parts:
- added G***: LOGO, TIH:electronic_cats_logo_8x6, F.Cu at (131.3, 100.8)
- added REF***: OSHW-Logo2_7.3x6mm_SilkScreen, Symbols:OSHW-Logo2_7.3x6mm_SilkScreen, F.Cu at (120.4, 100.3)
- P2: value - INPUT 12 + -> -INPUT12+
- P4: value Battery -> -Battery+
- U4: value RFM95W-868S2 -> RFM95W
